Commit message: Lidar,camera and depth camera added

File: description/robot.urdf.xacro (robot description, xacro)
@@ -3,3 +3,7 @@
     <!-- Example link -->
     <xacro:include filename="robot_core.xacro" />
+    <xacro:include filename="gazebo_control.xacro"/>
+    <xacro:include filename="lidar.xacro" />
+    <!-- <xacro:include filename="camera.xacro" /> -->
+    <xacro:include filename="depth_camera.xacro" />
 </robot>

File: description/robot_core.xacro (robot description, xacro)
@@ -13,4 +13,7 @@
 <material name = "black">
   <color rgba="0 0 0 1"/>
+</material>
+<material name="red">
+    <color rgba="1 0 0 1"/>
 </material>
 <!-- BASE LINK-->
@@ -41,4 +44,7 @@
 </xacro:inertial_box>
 </link>
+<gazebo reference="chassis">
+    <material>Gazebo/White</material>
+</gazebo>
 <!-- LEFT WHEEL LINK-->
 <joint name="left_wheel_joint" type="continuous">
@@ -64,4 +70,7 @@
     </xacro:inertial_cylinder>
 </link>
+<gazebo reference="left_wheel">
+    <material>Gazebo/Blue</material>
+</gazebo>
 <!-- RIGHT WHEEL LINK -->
 <joint name="right_wheel_joint" type="continuous">
@@ -87,4 +96,7 @@
     </xacro:inertial_cylinder>
 </link>
+<gazebo reference="right_wheel">
+    <material>Gazebo/Blue</material>
+</gazebo>
  <!-- CASTER WHEEL LINK -->
  <joint name="caster_wheel_joint" type="fixed">
@@ -109,3 +121,8 @@
     </xacro:inertial_sphere>
 </link>
+<gazebo reference="caster_wheel">
+    <material>Gazebo/Black</material>
+    <mu1 value="000.1"/>
+    <mu2 value="000.1"/>
+</gazebo>
 </robot>

Commit message: Teleop and Slam-toolbox added

File: description/robot.urdf.xacro (robot description, xacro)
@@ -1,10 +1,16 @@
 <?xml version="1.0"?>
 <robot xmlns:xacro="http://www.ros.org/wiki/xacro"  name="robot">
-    <!-- Example link -->
+    <!-- <xacro:arg name="use_ros2_control" default="true"/>
+    <xacro:if value="$(arg use_ros2_control)">
+        <xacro:include filename="ros2_control.xacro" />
+    </xacro:if>
+    <xacro:unless value="$(arg use_ros2_control)">
+        <xacro:include filename="gazebo_control.xacro" />
+    </xacro:unless> -->
     <xacro:include filename="robot_core.xacro" />
     <!-- <xacro:include filename="gazebo_control.xacro"/> -->
     <xacro:include filename="ros2_control.xacro"/>
     <xacro:include filename="lidar.xacro" />
-    <!-- <xacro:include filename="camera.xacro" /> -->
     <xacro:include filename="depth_camera.xacro" />
+     <!-- <xacro:include filename="camera.xacro" /> -->
 </robot>

File: description/robot_core.xacro (robot description, xacro)
@@ -19,4 +19,12 @@
 <!-- BASE LINK-->
 <link name="base_link">
+</link>
+<!-- BASE_FOOTPRINT LINK -->
+<joint name="base_footprint_joint" type="fixed">
+    <parent link="base_link"/>
+    <child link="base_footprint"/>
+    <origin xyz="0 0 0" rpy="0 0 0"/>
+</joint>
+<link name="base_footprint">
 </link>
 <!-- CHASSIS LINK-->
@@ -57,5 +65,5 @@
     <visual>
         <geometry>
-            <cylinder radius="0.05" length="0.04"/>
+            <sphere radius="0.05"/>
         </geometry>
         <material name="blue"/>
@@ -82,6 +90,6 @@
 <link name="right_wheel">
     <visual>
-        <geometry>
-            <cylinder radius="0.05" length="0.04"/>
+         <geometry>
+            <sphere radius="0.05"/>
         </geometry>
         <material name="blue"/>
