Commit message: Added package , some logging capabilities and quality of life changes

File: description/imu.xacro (robot description, xacro)
@@ -27,5 +27,5 @@
     <!--JOINTS-->
     <joint name="base_imu_joint" type="fixed">
-        <parent link="base_link" />
+        <parent link="chassis" />
         <child link="imu_link" />
         <origin xyz="0 0 0" rpy="0 0 0" />

File: description/lidar.xacro (robot description, xacro)
@@ -26,5 +26,5 @@
         <sensor name="laser" type="ray">
             <pose> 0 0 0 0 0 0 </pose>
-            <visualize>false</visualize>
+            <visualize>true</visualize>
             <update_rate>10</update_rate>
             <ray>
@@ -36,13 +36,13 @@
                         <max_angle>3.14</max_angle>
                     </horizontal>
-                    <vertical>
+                    <!-- <vertical>
                         <samples>90</samples>
                         <resolution>1</resolution>
                         <min_angle>-0.785</min_angle>
                         <max_angle>0.785</max_angle>
-                    </vertical>
+                    </vertical> -->
                 </scan>
                 <range>
-                    <min>0.35</min>
+                    <min>0.07</min> <!-- 0.35 (Original)-->
                     <max>12</max>
                     <resolution>0.03</resolution>
@@ -50,9 +50,9 @@
             </ray>
             <plugin name="laser_controller" filename="libgazebo_ros_ray_sensor.so">
-                <!-- <ros>
+                <ros>
                     <argument>~/out:=scan</argument>
-                </ros> -->
-                <output_type>sensor_msgs/PointCloud2</output_type>
-                <!-- <output_type>sensor_msgs/LaserScan</output_type> -->
+                </ros>
+                <!-- <output_type>sensor_msgs/PointCloud2</output_type> -->
+                <output_type>sensor_msgs/LaserScan</output_type>
                 <frame_name>laser_frame</frame_name>
             </plugin>

File: description/robot.urdf.xacro (robot description, xacro)
@@ -12,6 +12,6 @@
     <xacro:include filename="ros2_control.xacro"/>
     <xacro:include filename="lidar.xacro" />
-    <xacro:include filename="imu.xacro" />
-    <xacro:include filename="depth_camera.xacro" />
+    <!-- <xacro:include filename="imu.xacro" /> -->
+    <!-- <xacro:include filename="depth_camera.xacro" /> -->
      <!-- <xacro:include filename="camera.xacro" /> -->
 </robot>

Commit message: Added skid steering model, added velodyne

File: description/imu.xacro (robot description, xacro)
@@ -1,25 +1,23 @@
 <?xml version="1.0"?>
-<robot xmlns:xacro="http://www.ros.org/wiki/xacro" >
+<robot xmlns:xacro="http://www.ros.org/wiki/xacro">
     <!--IMU_MODEL____________________________________________________________________-->
-    <!--MATERIALS-->
-    <!-- <xacro:_make_colour colour="Red" rgb="1 0 0"/> -->
     <!--LINKS-->
     <link name="imu_link">
         <inertia>
-           <origin xyz="0 0 0" rpy="0 0 0" />
+            <origin xyz="0 0 0" rpy="0 0 0" />
             <mass value="0.1" />
             <inertia ixx="1" ixy="0.0" ixz="0.0" iyy="1" iyz="0.0" izz="1" />
         </inertia>
         <visual>
+            <origin xyz="0 0 0" rpy="0 0 0" />
             <geometry>
-                <cylinder radius="0.05" length="0.04" />
+                <box size="0.04 0.04 0.02" /> <!-- length x width x height -->
             </geometry>
-            <origin xyz="0 0 0" rpy="0 0 0" />
-            <material name="red" />
+            <material name="orange" />
         </visual>
         <collision>
             <origin xyz="0 0 0" rpy="0 0 0" />
             <geometry>
-                <cylinder radius="0.05" length="0.04" />
+                <box size="0.04 0.04 0.02" />
             </geometry>
         </collision>
@@ -29,29 +27,30 @@
         <parent link="chassis" />
         <child link="imu_link" />
-        <origin xyz="0 0 0" rpy="0 0 0" />
+        <origin xyz="0.1 0 0.205" rpy="0 0 0" />
     </joint>
     <!--SENSOR-->
     <gazebo reference="imu_link">
+        <material>Gazebo/orange</material>
         <gravity>true</gravity>
         <sensor name="imu_sensor" type="imu">
-          <always_on>true</always_on>
-          <update_rate>100</update_rate>
-          <visualize>true</visualize>
-          <topic>__default_topic__</topic>
-          <plugin filename="libgazebo_ros_imu_sensor.so" name="imu_plugin">
-            <topicName>imu</topicName>
-            <bodyName>imu_link</bodyName>
-            <updateRateHZ>10.0</updateRateHZ>
-            <gaussianNoise>0.0</gaussianNoise>
-            <xyzOffset>0 0 0</xyzOffset>
-            <rpyOffset>0 0 0</rpyOffset>
-            <frameName>imu_link</frameName>
-            <initialOrientationAsReference>false</initialOrientationAsReference>
-            <!-- <ros>
+            <always_on>true</always_on>
+            <update_rate>100</update_rate>
+            <visualize>true</visualize>
+            <topic>__default_topic__</topic>
+            <plugin filename="libgazebo_ros_imu_sensor.so" name="imu_plugin">
+                <topicName>imu</topicName>
+                <bodyName>imu_link</bodyName>
+                <updateRateHZ>10.0</updateRateHZ>
+                <gaussianNoise>0.0</gaussianNoise>
+                <xyzOffset>0 0 0</xyzOffset>
+                <rpyOffset>0 0 0</rpyOffset>
+                <frameName>imu_link</frameName>
+                <initialOrientationAsReference>false</initialOrientationAsReference>
+                <!-- <ros>
                 <remapping>${namespace}_imu_plugin/out:=/${namespace}_imu_plugin/out</remapping>
-            </ros> -->
-          </plugin>
-          <pose>0 0 0 0 0 0</pose>
+                </ros> -->
+            </plugin>
+            <pose>0 0 0 0 0 0</pose>
         </sensor>
-      </gazebo>
+    </gazebo>
 </robot>

File: description/lidar2D.xacro (robot description, xacro)
@@ -31,20 +31,22 @@
                 <scan>
                     <horizontal>
-                        <samples>360</samples>
-                        <resolution>1</resolution>
-                        <min_angle>-3.14</min_angle>
-                        <max_angle>3.14</max_angle>
+                        <!--Full lidar-->
+                        <!-- <samples>360</samples>
+                        <resolution>1</resolution> -->
+                        <!-- Real lidar-->
+                        <samples>1081</samples>
+                        <resolution>0.25</resolution>
+                        <!-- 360-->
+                        <!-- <min_angle>-3.14159</min_angle>
+                        <max_angle>3.14159</max_angle> -->
+                        <!--135-->
+                        <min_angle>-2,35619</min_angle>
+                        <max_angle>2,35619</max_angle>
                     </horizontal>
-                    <!-- <vertical>
-                        <samples>90</samples>
-                        <resolution>1</resolution>
-                        <min_angle>-0.785</min_angle>
-                        <max_angle>0.785</max_angle>
-                    </vertical> -->
                 </scan>
                 <range>
                     <min>0.07</min> <!-- 0.35 (Original)-->
                     <max>12</max>
-                    <resolution>0.03</resolution>
+                    <resolution>0.01</resolution>
                 </range>
             </ray>
@@ -53,5 +55,4 @@
                     <argument>~/out:=scan</argument>
                 </ros>
-                <!-- <output_type>sensor_msgs/PointCloud2</output_type> -->
                 <output_type>sensor_msgs/LaserScan</output_type>
                 <frame_name>laser_frame</frame_name>

File: description/lidar3D.xacro (robot description, xacro)
@@ -31,20 +31,20 @@
                 <scan>
                     <horizontal>
-                        <samples>360</samples>
+                        <samples>1800</samples>          <!-- VLP-16 1800 / Other 360-->
                         <resolution>1</resolution>
-                        <min_angle>-3.14</min_angle>
-                        <max_angle>3.14</max_angle>
+                        <min_angle>-3.14159</min_angle>
+                        <max_angle>3.14159</max_angle>
                     </horizontal>
                     <vertical>
-                        <samples>90</samples>
+                        <samples>16</samples>           <!-- VLP-16 16 / Other 90-->
                         <resolution>1</resolution>
-                        <min_angle>-0.785</min_angle>
-                        <max_angle>0.785</max_angle>
+                        <min_angle>-0.2618</min_angle>   <!-- VLP-16 -0.2618 / Other -0.785 -->
+                        <max_angle>0.2618</max_angle>    <!-- VLP-16 +0.2618 / Other +0.785)-->
                     </vertical>
                 </scan>
                 <range>
-                    <min>0.07</min> <!-- 0.35 (Original)-->
-                    <max>12</max>
-                    <resolution>0.03</resolution>
+                    <min>0.1</min> <!-- VLP-16 0.1)-->
+                    <max>100</max>   <!-- VLP-16 100)-->
+                    <resolution>0.01</resolution>
                 </range>
             </ray>

File: description/robot.urdf.xacro (robot description, xacro)
@@ -9,10 +9,13 @@
     </xacro:unless> -->
     <xacro:include filename="robot_core.xacro" />
+    <!-- <xacro:include filename="husky_core.xacro" /> -->
     <!-- <xacro:include filename="gazebo_control.xacro"/> -->
     <xacro:include filename="ros2_control.xacro"/>
-    <xacro:include filename="lidar2D.xacro" />
-    <!-- <xacro:include filename="lidar3D.xacro" /> -->
-    <!-- <xacro:include filename="imu.xacro" /> -->
+    <!-- <xacro:include filename="ros2_control_husky.xacro"/> -->
+    <!-- <xacro:include filename="lidar2D.xacro" /> -->
+    <xacro:include filename="lidar3D.xacro" />
+    <!-- <xacro:include filename="lidar_VLP16.xacro" /> -->
+    <xacro:include filename="imu.xacro" />
     <!-- <xacro:include filename="depth_camera.xacro" /> -->
-     <!-- <xacro:include filename="camera.xacro" /> -->
+    <!-- <xacro:include filename="camera.xacro" /> -->
 </robot>
