Commit message: 3D slam starting to to work, husky with rotating llidar urdf ready

File: description/husky_core.xacro (robot description, xacro)
@@ -9,4 +9,10 @@
         <color rgba="1 1 0 1"/>
     </material>
+    <material name="orange">
+        <color rgba="1 0.5 0 1"/>
+    </material>
+    <material name="blue">
+        <color rgba="0 0 1 1"/>
+    </material>
     <material name="black">
         <color rgba="0 0 0 1"/>
@@ -14,4 +20,7 @@
     <material name="red">
         <color rgba="1 0 0 1"/>
+    </material>
+    <material name="grey">
+        <color rgba="0.5 0.5 0.5 1" />
     </material>
     <!-- BASE LINK -->

File: description/imu.xacro (robot description, xacro)
@@ -31,5 +31,5 @@
     <!--SENSOR-->
     <gazebo reference="imu_link">
-        <material>Gazebo/orange</material>
+        <material>Gazebo/Orange</material>
         <gravity>true</gravity>
         <sensor name="imu_sensor" type="imu">

File: description/lidar2D.xacro (robot description, xacro)
@@ -1,8 +1,13 @@
 <?xml version="1.0"?>
 <robot xmlns:xacro="http://www.ros.org/wiki/xacro">
-    <joint name="laser_joint" type="fixed">
+    <!-- <joint name="laser_joint" type="fixed">
         <parent link="chassis" />
         <child link="laser_frame" />
         <origin xyz="0.1 0 0.175" rpy="0 0 0" />
+    </joint> -->
+    <joint name="laser_joint" type="fixed">
+        <parent link="base_link" />
+        <child link="laser_frame" />
+        <origin xyz="0.4 0 0.5" rpy="0 0 0" />
     </joint>
     <link name="laser_frame">

File: description/lidar3D.xacro (robot description, xacro)
@@ -1,8 +1,13 @@
 <?xml version="1.0"?>
 <robot xmlns:xacro="http://www.ros.org/wiki/xacro">
-    <joint name="laser_joint" type="fixed">
+    <!-- <joint name="laser_joint" type="fixed">
         <parent link="chassis" />
         <child link="laser_frame" />
         <origin xyz="0.1 0 0.4" rpy="0 0 0" />
+    </joint> -->
+    <joint name="laser_joint" type="fixed">
+        <parent link="base_link" />
+        <child link="laser_frame" />
+        <origin xyz="0.4 0 0.5" rpy="0 0 0" />
     </joint>
     <link name="laser_frame">

File: description/lidar_VLP16.xacro (robot description, xacro)
@@ -6,8 +6,13 @@
         <child link="velodyne_base_link" />
     </joint> -->
-    <joint name="velodyne_base_mount_joint" type="fixed">
+    <!-- <joint name="velodyne_base_mount_joint" type="fixed">
         <parent link="chassis" />
         <child link="velodyne_base_link" />
-        <origin xyz="0.1 0 0.4" rpy="0 0 0" />
+        <origin xyz="0.0 0 0.4" rpy="0 0 0" />
+    </joint> -->
+    <joint name="velodyne_base_mount_joint" type="fixed">
+        <parent link="base_link" />
+        <child link="velodyne_base_link" />
+        <origin xyz="0.4 0 0.5" rpy="0 0 0" />
     </joint>
     <!-- <link name="velodyne_base_link">
@@ -86,4 +91,5 @@
     <!-- Gazebo requires the velodyne_gazebo_plugins package -->
     <gazebo reference="velodyne">
+        <material>Gazebo/Red</material>
         <sensor name="velodyne-VLP16" type="ray">
             <pose>0 0 0 0 0 0</pose>

File: description/robot.urdf.xacro (robot description, xacro)
@@ -8,11 +8,11 @@
         <xacro:include filename="gazebo_control.xacro" />
     </xacro:unless> -->
-    <xacro:include filename="robot_core.xacro" />
-    <!-- <xacro:include filename="husky_core.xacro" /> -->
+    <!-- <xacro:include filename="robot_core.xacro" /> -->
+    <xacro:include filename="husky_core.xacro" />
     <!-- <xacro:include filename="gazebo_control.xacro"/> -->
-    <xacro:include filename="ros2_control.xacro"/>
-    <!-- <xacro:include filename="ros2_control_husky.xacro"/> -->
+    <!-- <xacro:include filename="ros2_control.xacro"/> -->
+    <xacro:include filename="ros2_control_husky.xacro"/>
     <!-- <xacro:include filename="lidar2D.xacro" /> -->
-    <xacro:include filename="lidar3D.xacro" />
+    <!-- <xacro:include filename="lidar3D.xacro" /> -->
     <!-- <xacro:include filename="lidar_VLP16.xacro" /> -->
     <xacro:include filename="imu.xacro" />

File: description/ros2_control_husky.xacro (robot description, xacro)
@@ -41,4 +41,5 @@
         <plugin name="gazebo_ros2_control" filename="libgazebo_ros2_control.so">
             <parameters>$(find my_bot)/config/my_controllers_husky.yaml</parameters>
+            <!-- <robot_param_node>my_bot</robot_param_node> -->
         </plugin>
     </gazebo>
