Commit message: Small stuff

File: description/lidar2D.xacro (robot description, xacro)
@@ -9,5 +9,6 @@
         <parent link="base_link" />
         <child link="laser_frame" />
-        <origin xyz="0.4 0 0.5" rpy="0 0 0" />
+        <!-- <origin xyz="0.4 0 0.5" rpy="0 0 0" /> -->
+        <origin xyz="0.0 0 0.5" rpy="0 0 0" />
     </joint>
     <link name="laser_frame">
@@ -29,7 +30,7 @@
     <gazebo reference="laser_frame">
         <material>Gazebo/Red</material>
-        <sensor name="laser" type="ray">
+        <sensor name="laser_front" type="ray">
             <pose> 0 0 0 0 0 0 </pose>
-            <visualize>true</visualize>
+            <visualize>false</visualize>
             <update_rate>10</update_rate>
             <ray>
@@ -46,6 +47,6 @@
                         <max_angle>3.14159</max_angle> -->
                         <!--135-->
-                        <min_angle>-2,35619</min_angle>
-                        <max_angle>2,35619</max_angle>
+                        <min_angle>-2.35619</min_angle>
+                        <max_angle>2.35619</max_angle>
                     </horizontal>
                 </scan>
@@ -56,5 +57,5 @@
                 </range>
             </ray>
-            <plugin name="laser_controller" filename="libgazebo_ros_ray_sensor.so">
+            <plugin name="laser_controller_front" filename="libgazebo_ros_ray_sensor.so">
                 <ros>
                     <argument>~/out:=scan</argument>

File: description/lidar_VLP16.xacro (robot description, xacro)
@@ -14,5 +14,5 @@
         <parent link="base_link" />
         <child link="velodyne_base_link" />
-        <origin xyz="0.4 0 0.5" rpy="0 0 0" />
+        <origin xyz="0.0 0 0.5" rpy="0 0 0" />
     </joint>
     <!-- <link name="velodyne_base_link">

File: description/robot.urdf.xacro (robot description, xacro)
@@ -15,5 +15,5 @@
     <!-- <xacro:include filename="lidar2D.xacro" /> -->
     <!-- <xacro:include filename="lidar3D.xacro" /> -->
-    <!-- <xacro:include filename="lidar_VLP16.xacro" /> -->
+    <xacro:include filename="lidar_VLP16.xacro" />
     <xacro:include filename="imu.xacro" />
     <!-- <xacro:include filename="depth_camera.xacro" /> -->

File: description/robot_and_lidar.urdf.xacro (robot description, xacro)
@@ -4,4 +4,5 @@
     <xacro:include filename="husky_core.xacro" />
     <xacro:include filename="imu.xacro" />
+    <xacro:include filename="lidar2D.xacro" />
     <xacro:include filename="$(find my_bot)/description/lidar_husky_control_gazebo.xacro" />
     <joint name="husky_lidar_joint" type="fixed">
